Commit message: multiple robots added

File: projects/devel/webots_ros2_suv/resource/suv1.urdf (robot description, URDF)
Before this commit: robot /home/hiber/Downloads/suv.urdf, 23 links, 24 joints
Links:
- added link compass
- added link gps
- added link inertial unit
- added link left_wing_camera
- added link lidar
- added link range_finder
Joints:
- added joint base_link_camera_left_joint: type fixed, parent base_link, child left_wing_camera, origin xyz=1.73 0 1.38 rpy=-1.570796 0 -1.570796
- added joint base_link_compass_joint: type fixed, parent base_link, child compass, origin xyz=1 0 1.45 rpy=0 0 0
- added joint base_link_gps_joint: type fixed, parent base_link, child gps, origin xyz=1 0 1.45 rpy=0 0 0
- added joint base_link_inertial unit_joint: type fixed, parent base_link, child inertial unit, origin xyz=1 0 1.45 rpy=0 0 0
- added joint base_link_lidar_joint: type fixed, parent base_link, child lidar, origin xyz=1 0 1.45 rpy=0 0 0
- added joint base_link_range_finder_joint: type fixed, parent base_link, child range_finder, origin xyz=1.73 0 1.38 rpy=-1.570796 0 -1.570796
- joint base_link_Velodyne HDL-64E_joint: origin xyz=1 0 1.61 rpy=-0.000007 -0.000007 3.14159 -> xyz=1 0 1.63 rpy=0 0 0
- joint base_link_camera_joint: origin xyz=3.85 0 0.45 rpy=-1.570796 0 -1.570796 -> xyz=1.73 0 1.38 rpy=-1.570796 0 -1.570796
- joint left_rear_sensor: origin xyz=0.001434 0.812566 0 rpy=2.095027 0 -1.5708 -> xyz=0 0.814 0 rpy=0 0 -1.5708
- joint right_rear_sensor: origin xyz=0.001434 -0.812566 0 rpy=-1.532408 0 1.5708 -> xyz=0 -0.814 0 rpy=0 0 1.5708
- joint slot_1_rear left wheel_joint: origin xyz=-0.001434 0.096746 -0.055938 rpy=0 0 0 -> xyz=0 0 0 rpy=0 0 0
- joint slot_rear right wheel_joint: origin xyz=-0.001434 -0.111671 0.004289 rpy=0 0 0 -> xyz=0 0 0 rpy=0 0 0
